Commit message: Fix base_link -> chassis

File: simulation_ws/src/robot_bringup/description/lidar.xacro (robot description, xacro)
@@ -20,5 +20,5 @@
     </link>
     <joint name="laser_joint" type="fixed">
-        <parent link="base_link"/>
+        <parent link="chassis"/>
         <child link="laser_frame"/>
         <origin xyz="0 0 0.205" rpy="0 0 0"/>

File: simulation_ws/src/robot_bringup/description/swarm_bot.urdf (robot description, URDF)
Before this commit: robot swarm_bot, 7 links, 6 joints
Links:
- removed link base_link
- added link chassis, mass 0.5; collision cylinder length=0.15 radius=0.107; visual cylinder length=0.15 radius=0.107
Joints:
- joint laser_joint: parent base_link -> chassis
- joint origin_joint: child base_link -> chassis

File: simulation_ws/src/robot_bringup/description/swarm_bot.xacro (robot description, xacro)
@@ -9,5 +9,5 @@
     </link>
     <!-- Base -->
-    <link name="base_link">
+    <link name="chassis">
         <visual>
             <!-- change the position of the visualization only, not the axis -->
@@ -31,5 +31,5 @@
         </xacro:inertial_cylinder>
     </link>
-    <gazebo reference="base_link">
+    <gazebo reference="chassis">
         <material>Gazebo/White</material>
     </gazebo>
@@ -131,5 +131,5 @@
     <joint name="origin_joint" type="fixed">
         <parent link="origin_link"/>
-        <child link="base_link"/>
+        <child link="chassis"/>
         <origin xyz="0 0 -0.0325"/>
     </joint>
