Commit message: Fix origin_link -> base_link

File: simulation_ws/src/robot_bringup/description/gazebo_control.xacro (robot description, xacro)
@@ -19,5 +19,5 @@
             <!-- Output -->
             <odometry_frame>odom</odometry_frame>
-            <robot_base_frame>origin_link</robot_base_frame>
+            <robot_base_frame>base_link</robot_base_frame>
             <publish_odom>true</publish_odom>
             <publish_odom_tf>true</publish_odom_tf>

File: simulation_ws/src/robot_bringup/description/swarm_bot.urdf (robot description, URDF)
Before this commit: robot swarm_bot, 7 links, 6 joints
Links:
- removed link origin_link
- added link base_link
Joints:
- joint back_passive_wheel_joint: parent origin_link -> base_link
- joint front_passive_wheel_joint: parent origin_link -> base_link
- joint left_wheel_joint: parent origin_link -> base_link
- joint origin_joint: parent origin_link -> base_link
- joint right_wheel_joint: parent origin_link -> base_link

File: simulation_ws/src/robot_bringup/description/swarm_bot.xacro (robot description, xacro)
@@ -6,5 +6,5 @@
     <!-- LINKS -->
     <!-- Origin -->
-    <link name="origin_link">
+    <link name="base_link">
     </link>
     <!-- Base -->
@@ -130,5 +130,5 @@
     <!-- Base -->
     <joint name="origin_joint" type="fixed">
-        <parent link="origin_link"/>
+        <parent link="base_link"/>
         <child link="chassis"/>
         <origin xyz="0 0 -0.0325"/>
@@ -136,5 +136,5 @@
     <!-- Left Wheel -->
     <joint name="right_wheel_joint" type="continuous">
-        <parent link="origin_link"/>
+        <parent link="base_link"/>
         <child link="right_wheel"/>
         <!-- rotate wheel 90 deg around x-axis -->
@@ -144,5 +144,5 @@
     <!-- Right Wheel -->
     <joint name="left_wheel_joint" type="continuous">
-        <parent link="origin_link"/>
+        <parent link="base_link"/>
         <child link="left_wheel"/>
         <origin xyz="0 0.107 0" rpy="${pi/2} 0 0"/>
@@ -151,5 +151,5 @@
     <!-- Front Passive Wheel -->
     <joint name="front_passive_wheel_joint" type="fixed">
-        <parent link="origin_link"/>
+        <parent link="base_link"/>
         <child link="front_passive_wheel"/>
         <origin xyz="0.067 0 -0.0085" rpy="0 0 0"/>
@@ -157,5 +157,5 @@
     <!-- Back Passive Wheel -->
     <joint name="back_passive_wheel_joint" type="fixed">
-        <parent link="origin_link"/>
+        <parent link="base_link"/>
         <child link="back_passive_wheel"/>
         <origin xyz="-0.067 0 -0.0083" rpy="0 0 0"/>
