Commit message: Fix base_link -> chassis

File: simulation_ws/src/install/robot_bringup/share/robot_bringup/description/swarm_bot.urdf (robot description, URDF)
Before this commit: robot swarm_bot, 7 links, 6 joints
Links:
- removed link base_link
- added link chassis, mass 0.5; collision cylinder length=0.15 radius=0.107; visual cylinder length=0.15 radius=0.107
Joints:
- joint laser_joint: parent base_link -> chassis
- joint origin_joint: child base_link -> chassis

File: simulation_ws/src/robot_bringup/description/gazebo_control.xacro (robot description, xacro)
@@ -5,8 +5,8 @@
         <plugin name="diff_drive_controller" filename="libgazebo_ros_diff_drive.so">
             <!-- ROS parameters -->
-            <ros>
+            <!-- <ros>
                 <namespace>robot_namespace</namespace>
                 <param name="robot_description" value="robot_description" />
-            </ros>
+            </ros> -->
             <!-- Wheel Information -->
             <left_joint>left_wheel_joint</left_joint>
