Commit message: Fix origin_link -> base_link

File: simulation_ws/src/install/robot_bringup/share/robot_bringup/description/gazebo_control.xacro (robot description, xacro)
@@ -19,5 +19,5 @@
             <!-- Output -->
             <odometry_frame>odom</odometry_frame>
-            <robot_base_frame>origin_link</robot_base_frame>
+            <robot_base_frame>base_link</robot_base_frame>
             <publish_odom>true</publish_odom>
             <publish_odom_tf>true</publish_odom_tf>

File: simulation_ws/src/install/robot_bringup/share/robot_bringup/description/swarm_bot.urdf (robot description, URDF)
Before this commit: robot swarm_bot, 7 links, 6 joints
Links:
- removed link origin_link
- added link base_link
Joints:
- joint back_passive_wheel_joint: parent origin_link -> base_link
- joint front_passive_wheel_joint: parent origin_link -> base_link
- joint left_wheel_joint: parent origin_link -> base_link
- joint origin_joint: parent origin_link -> base_link
- joint right_wheel_joint: parent origin_link -> base_link
